Commit message: Fix URDF wheel position (flip to opposite side), add per-motor speed trim

File: scripts/robot.urdf (robot description, URDF)
Before this commit: robot soccer_bot, 6 links, 5 joints
Joints:
- joint chassis_to_left_wheel: origin xyz=-0.115 0.105 0.033 rpy=-1.5708 0 0 -> xyz=0.115 0.105 0.033 rpy=-1.5708 0 0
- joint chassis_to_right_wheel: origin xyz=-0.115 -0.105 0.033 rpy=-1.5708 0 0 -> xyz=0.115 -0.105 0.033 rpy=-1.5708 0 0

Commit message: Add rosboard and soccer bot updates

File: scripts/robot.urdf (robot description, URDF)
Before this commit: robot soccer_bot, 6 links, 5 joints
Joints:
- joint base_to_chassis: origin xyz=0 0 0 -> xyz=0 0 0 rpy=0 0 0
- joint chassis_to_left_wheel: origin xyz=0.115 0.105 0.033 rpy=-1.5708 0 0 -> xyz=-0.115 0.105 0.033 rpy=-1.5708 0 0
- joint chassis_to_right_wheel: origin xyz=0.115 -0.105 0.033 rpy=-1.5708 0 0 -> xyz=-0.115 -0.105 0.033 rpy=-1.5708 0 0

Commit message: feat(rviz): integrate 4-DOF robotic arm URDF, live joint states, dynamic TF and enable SLAM map and path in RViz2

File: scripts/robot.urdf (robot description, URDF)
Before this commit: robot soccer_bot, 6 links, 5 joints
Links:
- added link arm_base_link; visual cylinder length=0.03 radius=0.032
- added link arm_elbow_link; visual cylinder length=0.10 radius=0.011
- added link arm_left_claw; visual box size=0.06 0.008 0.02
- added link arm_mount; visual cylinder length=0.015 radius=0.04
- added link arm_right_claw; visual box size=0.06 0.008 0.02
- added link arm_shoulder_link; visual cylinder length=0.10 radius=0.012
- added link arm_wrist_link; visual box size=0.03 0.04 0.025
Joints:
- added joint base_joint: type revolute, parent arm_mount, child arm_base_link, origin xyz=0 0 0.015 rpy=0 0 0, axis 0 0 1, limit lower=-1.5708 upper=1.5708 effort=10.0 velocity=3.0
- added joint chassis_to_arm_mount: type fixed, parent chassis, child arm_mount, origin xyz=0.10 0.0 0.11 rpy=0 0 0
- added joint elbow_joint: type revolute, parent arm_shoulder_link, child arm_elbow_link, origin xyz=0 0 0.10 rpy=0 0 0, axis 0 1 0, limit lower=-1.5708 upper=2.6179 effort=10.0 velocity=3.0
- added joint gripper_left_joint: type revolute, parent arm_wrist_link, child arm_left_claw, origin xyz=0.025 0.015 0 rpy=0 0 0, axis 0 0 1, limit lower=0.0 upper=0.8 effort=5.0 velocity=3.0
- added joint gripper_right_joint: type revolute, parent arm_wrist_link, child arm_right_claw, origin xyz=0.025 -0.015 0 rpy=0 0 0, axis 0 0 -1, limit lower=0.0 upper=0.8 effort=5.0 velocity=3.0
- added joint shoulder_joint: type revolute, parent arm_base_link, child arm_shoulder_link, origin xyz=0 0 0.03 rpy=0 0 0, axis 0 1 0, limit lower=-0.5 upper=2.6179 effort=10.0 velocity=3.0
- added joint wrist_joint: type fixed, parent arm_elbow_link, child arm_wrist_link, origin xyz=0.10 0 0 rpy=0 0 0
